File: T2601_APIArduino_MezaDivider/T2601_APIArduino_MezaDivider.kicad_sch (KiCad schematic)
At the start: 27 parts, among them J1 Conn_01x10, J2 Conn_01x10

Commit message: Mezza Divider V1
Parts:
- removed R1, R2, R3, R4, R5, R6, R7, R8: 7.5kΩ, PCM_JLCPCB:R_0603, symbol PCM_JLCPCB-Resistors:0603,7.5kΩ
- removed R10, R11, R12, R13, R14, R15, R16, R9: 5.1kΩ, PCM_JLCPCB:R_0603, symbol PCM_JLCPCB-Resistors:0603,5.1kΩ
- added R1, R2, R3, R4, R5, R6, R7, R8: 15kΩ, PCM_JLCPCB:R_0402, symbol PCM_JLCPCB-Resistors:0402,15kΩ
- added R10, R11, R12, R13, R14, R15, R16, R9: 10kΩ, PCM_JLCPCB:R_0402, symbol PCM_JLCPCB-Resistors:0402,10kΩ
Connections:
- net 1: now also R1.2, R9.1
- net 2: now also R10.1, R2.2
- net 3: now also R11.1, R3.2
- net 4: now also R12.1, R4.2
- net 5: now also R13.1, R5.2
- net 6: now also R14.1, R6.2
- net 7: now also R15.1, R7.2
- net 8: now also R16.1, R8.2
- net GND: now also R10.2, R11.2, R12.2, R13.2, R14.2, R15.2, R16.2, R9.2
- net OUT_1: now also R1.1
- net OUT_2: now also R2.1
- net OUT_3: now also R3.1
- net OUT_4: now also R4.1
- net OUT_5: now also R5.1
- net OUT_6: now also R6.1
- net OUT_7: now also R7.1
- net OUT_8: now also R8.1
