File: T2601_APIArduino_MezaDivider/T2601_APIArduino_MezaDivider.kicad_pcb (KiCad board)
At the start: 2 copper layers, 26.4 x 29 mm, 27 parts, among them J1 Conn_01x10, J2 Conn_01x10

Commit message: Mezza Divider V1
Parts:
- R1, R2, R3, R4, R5, R6, R7, R8: value 7.5kΩ -> 15kΩ; footprint PCM_JLCPCB:R_0603 -> PCM_JLCPCB:R_0402
- R10, R11, R12, R13, R14, R15, R16, R9: value 5.1kΩ -> 10kΩ; footprint PCM_JLCPCB:R_0603 -> PCM_JLCPCB:R_0402
- moved JP3 4.83 mm to (169.5, 92.9)
- moved JP1 4.82 mm to (174.6, 92.9)
- moved JP2 4.82 mm to (172.1, 92.9)
- moved JP4 4.82 mm to (167.0, 92.9)
- moved JP8 4.75 mm to (151.8, 92.9)
- moved JP7 4.74 mm to (154.3, 92.9)
- moved JP6 4.72 mm to (156.8, 92.9)
- moved JP5 4.72 mm to (159.4, 92.9)
- moved R8 1.08 mm to (151.8, 88.9), turned to 0 degrees
- moved R2 1.08 mm to (172.1, 88.9), turned to 180 degrees
- moved R1 1.05 mm to (174.7, 88.8), turned to 180 degrees
- moved R7 1.00 mm to (154.3, 88.9), turned to 0 degrees
- moved R5 0.98 mm to (159.4, 88.9), turned to 0 degrees
- moved R3 0.97 mm to (169.6, 88.9), turned to 180 degrees
- moved R4 0.97 mm to (167.0, 88.9), turned to 180 degrees
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Routing:
- net 8: track 16.4 -> 9.95 mm
- net 7: track 16.2 -> 9.97 mm
- net 2: track 15.8 -> 10.0 mm
- net 1: track 15.9 -> 10.1 mm
- net 6: track 15.6 -> 9.97 mm
- net 5: track 15.6 -> 10.0 mm
- net 4: track 14.5 -> 10.0 mm
- net 3: track 14.4 -> 9.98 mm
- net GND: track 10.1 -> 8.12 mm
- net OUT_1: track 19.4 -> 20.8 mm, vias 2 -> 0
- net OUT_8: track 19.2 -> 20.3 mm, vias 2 -> 0
- net OUT_2: track 19.2 -> 20.3 mm, vias 2 -> 0
- net OUT_6: track 19.3 -> 20.3 mm, vias 2 -> 0
- net OUT_3: track 19.3 -> 20.2 mm, vias 2 -> 0
- net OUT_7: track 19.3 -> 20.1 mm, vias 2 -> 0
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
Commit message: Meza Divider V1.1
Other:
- board text added: "Made on Earth by Humans"
- board text added: "T2601_APIArduino V1 Meza12VDivider JGY & DDP"
Changed lines of the file:
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@@
 		(layer "Edge.Cuts")
+	)
+	(gr_text "T2601_APIArduino\nV1 Meza12VDivider\nJGY & DDP"
+		(at 150.7998 99.9744 0)
+		(layer "F.SilkS")
+		(effects
+			(font
+				(size 1 1)
+				(thickness 0.25)
+				(bold yes)
+			)
+			(justify left bottom)
+		)
+	)
+	(gr_text "Made on Earth by Humans"
+		(at 173.6344 86.0044 0)
+		(layer "B.SilkS")
+		(effects
+			(font
+				(size 1 1)
+				(thickness 0.125)
+			)
+			(justify left bottom mirror)
+		)
 	)
 	(segment
