File: T2601_APIArduinoExtentionBoard/T2601_APIArduinoExtentionBoard.kicad_sch (KiCad schematic)
At the start: 98 parts, among them J1 Conn_01x10_Socket, J10 Conn_02x03_Counter_Clockwise, J11 Conn_01x04, J12 Screw_Terminal_01x02, J14 Screw_Terminal_01x02, J2 Conn_01x10_Socket, J20 Conn_02x08_Counter_Clockwise, J21 Conn_02x08_Counter_Clockwise, J3 Conn_01x10_Socket, J30 Conn_01x04_Pin, J31 Conn_01x04_Pin, J4 Conn_01x10_Socket, J5 Screw_Terminal_01x08, J6 Screw_Terminal_01x08, U2 ATmega328PB-A, X1 X322516MOB4SI

Commit message: Reorganisation schematic
Parts:
- removed C1, C2: 22pF, PCM_JLCPCB:C_0402, symbol PCM_JLCPCB-Capacitors:0402,22pF
- removed C3, C7, C8, C9: 100nF, PCM_JLCPCB:C_0402, symbol PCM_JLCPCB-Capacitors:0402,100nF
- removed D1: D_Schottky, Diode_THT:D_5W_P12.70mm_Horizontal, symbol Device:D_Schottky
- removed D10, D9: Yellow, PCM_JLCPCB:D_0805, symbol PCM_JLCPCB-Diodes:LED,0805,Yellow
- removed D26: Red, PCM_JLCPCB:D_0805, symbol PCM_JLCPCB-Diodes:LED,0805,Red
- removed D6: M7, PCM_JLCPCB:D_SMA, symbol PCM_JLCPCB-Diodes:General,M7
- removed J10: Conn_02x03_Counter_Clockwise, Connector_PinSocket_2.54mm:PinSocket_2x03_P2.54mm_Vertical, symbol Connector_Generic:Conn_02x03_Counter_Clockwise
- removed J11: Conn_01x04, Connector_PinSocket_2.54mm:PinSocket_1x04_P2.54mm_Vertical, symbol Connector_Generic:Conn_01x04
- removed R25, R6, R7: 1kΩ, PCM_JLCPCB:R_0402, symbol PCM_JLCPCB-Resistors:0402,1kΩ
- removed R5: 5.6kΩ, PCM_JLCPCB:R_0603, symbol PCM_JLCPCB-Resistors:0603,5.6kΩ
- removed S1: Tactile Button, 160gf, PCM_JLCPCB:SW-SMD_4P-L5.1-W5.1-P3.70-LS6.5-TL-2, symbol PCM_JLCPCB-Connectors_Buttons:Tactile Button, 160gf, 12V, 50mA, 5.1mm
- removed U2: ATmega328PB-A, Package_QFP:TQFP-32_7x7mm_P0.8mm, symbol MCU_Microchip_ATmega:ATmega328PB-A
- removed X1: X322516MOB4SI, T2601_APIArduinoExtentionBoard_Lib:CRYSTAL-SMD_4P-L3.2-W2.5-BL, symbol T2601_APIArduinoExtentionBoard_Lib:X322516MOB4SI
Other:
- added sheet T2601_APIArduinoExtentionBoard_Microcontroleur (T2601_APIArduinoExtentionBoard_Microcontroleur.kicad_sch)
- added sheet T2601_APIArduinoExtentionBoard_Programmation (T2601_APIArduinoExtentionBoard_Programmation.kicad_sch)
- note added: "Licence Copyright (C) 2026 HackHype This project is licensed under CERN OHL-S v2. See the LICENSE file for details."
- note removed: "Gen Reset"
- note removed: "License Copyright (C) 2026 HackHype This project is licensed under CERN OHL-S v2. See the LICENSE file for details."
- note removed: "PROG"
- note removed: "PROG Indicator"
- note removed: "Reset Indicator"
- note removed: "SERIAL debug"
- note removed: "TODO : Crystal Pin Prog Serial Blink Sur Pin Prog Schoky Diode prog C decouplage Led sur Serial Com Led Sur Serial Debug + prevoir Serial debug"
- note removed: "Tac Switch Reset"
- moved on the sheet: C5, C6, D11, D12, D14, D15, D16, D17, D18, D19, D2, D20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

Commit message: Nouveau schematic selon template V1
Parts:
- removed C5, C6: C, Capacitor_THT:C_Radial_D6.3mm_H11.0mm_P2.50mm, symbol Device:C
- removed D11, D12, D29: Yellow, PCM_JLCPCB:D_0805, symbol PCM_JLCPCB-Diodes:LED,0805,Yellow
- removed D14, D15, D16, D17, D18, D19, D2, D20, D21, D22, D23, D24, D25, D28, D3, D4, D5, D7, D8: Green, PCM_JLCPCB:D_0805, symbol PCM_JLCPCB-Diodes:LED,0805,Green
- removed D27: Red, PCM_JLCPCB:D_0805, symbol PCM_JLCPCB-Diodes:LED,0805,Red
- removed H1, H2, H3, H4: MountingHole, MountingHole:MountingHole_3.2mm_M3, symbol Mechanical:MountingHole
- removed J1, J2, J3, J4: Conn_01x10_Socket, Connector_PinSocket_2.54mm:PinSocket_1x10_P2.54mm_Vertical, symbol Connector:Conn_01x10_Socket
- removed J12, J14: Screw_Terminal_01x02, TerminalBlock:TerminalBlock_Xinya_XY308-2.54-2P_1x02_P2.54mm_Horizontal, symbol Connector:Screw_Terminal_01x02
- removed J20, J21: Conn_02x08_Counter_Clockwise, Connector_IDC:IDC-Header_2x08_P2.54mm_Vertical, symbol Connector_Generic:Conn_02x08_Counter_Clockwise
- removed J30, J31: Conn_01x04_Pin, Connector_JST:JST_XH_B4B-XH-A_1x04_P2.50mm_Vertical, symbol Connector:Conn_01x04_Pin
- removed J5, J6: Screw_Terminal_01x08, TerminalBlock_TE-Connectivity:TerminalBlock_TE_282834-8_1x08_P2.54mm_Horizontal, symbol Connector:Screw_Terminal_01x08
- removed JP1, JP10, JP11, JP12, JP2, JP3, JP4, JP5, JP6, JP7, JP8, JP9: SolderJumper_2_Open, Jumper:SolderJumper-2_P1.3mm_Open_RoundedPad1.0x1.5mm, symbol Jumper:SolderJumper_2_Open
- removed R1, R10, R11, R12, R13, R14, R15, R16, R17, R18, R19, R20, R21, R22, R26, R27, R28, R3, R4, R8, R9: 1kΩ, PCM_JLCPCB:R_0402, symbol PCM_JLCPCB-Resistors:0402,1kΩ
- removed R23: 2.4kΩ, PCM_JLCPCB:R_0603, symbol PCM_JLCPCB-Resistors:0603,2.4kΩ
- removed R24: 1kΩ, PCM_JLCPCB:R_0603, symbol PCM_JLCPCB-Resistors:0603,1kΩ
- removed TP1, TP2: TestPoint, TestPoint:TestPoint_Loop_D2.50mm_Drill1.0mm_LowProfile, symbol Connector:TestPoint
Connections:
- no-connect marks 4 -> 0
Other:
- removed sheet T2601_APIArduinoExtentionBoard_Microcontroleur
- removed sheet T2601_APIArduinoExtentionBoard_Programmation
- added sheet Block Diagram (T2601_Block Diagram.kicad_sch)
- added sheet Project Architecture (T2601_Project Architecture.kicad_sch)
- added sheet Revision History (T2601_Revision History.kicad_sch)
- note added: "${BOARD_NAME}"
- note added: "${CURRENT_DATE}"
- note added: "${VARIANT} ${RELEASE_DATE}"
- note added: "..........................................."
- note added: "1"
- note added: "10"
- note added: "11"
- note added: "12"
- note added: "13"
- note added: "14"
- note added: "15"
- note added: "16"
- note added: "17"
- note added: "18"
- note added: "19"
- note added: "2"
- note added: "20"
- note added: "21"
- note added: "22"
- note added: "23"
- note added: "24"
- note added: "25"
- note added: "26"
- note added: "27"
- note added: "28"
- note added: "29"
- note added: "3"
- note added: "30"
- note added: "31"
- note added: "32"
- note added: "33"
- note added: "34"
- note added: "35"
- note added: "36"
- note added: "37"
- note added: "38"
- note added: "39"
- note added: "4"
- note added: "40"
- note added: "5"
- note added: "6"
- note added: "7"
- note added: "8"
- note added: "9"
- note added: "Add a comment here"
- note added: "BOTTOM VIEW"
- note added: "Block Diagram"
- note added: "CHECKED - There shouldn't be any mistakes. Contact the engineer if you find any."
- note added: "Communication Bus"
- note added: "Cover Page"
- note added: "DESIGN CONSIDERATIONS"
- note added: "DRAFT - Very early stage of schematic, ignore details."
- note added: "Index"
- note added: "Licence Copyright (C) 2026 Jules Grucy This project is licensed under CERN OHL-S v2. See the LICENSE file for details."
- note added: "MCU"
- note added: "MCU I/O"
- note added: "MCU Programation"
- note added: "Miscellaneous"
- note added: "NOTES"
- note added: "Not fitted components are marked as"
- note added: "PRELIMINARY - Close to final schematic."
- note added: "Page"
- note added: "Power"
- note added: "Project Architecture"
- note added: "RELEASED - A board with this schematic has been sent to production."
- note added: "Rev ${REVISION}"
- note added: "Revision History"
- note added: "State: ${STATE}"
- note added: "TOP VIEW"
- note removed: "Conn PWR"
- note removed: "Conn Signal"
- note removed: "IO indicator"
- note removed: "Licence Copyright (C) 2026 HackHype This project is licensed under CERN OHL-S v2. See the LICENSE file for details."
- note removed: "Mezanine Connector & Output"
- note removed: "PWR Indicator"
- note removed: "SERIAL Indicator"
- note removed: "State Indicator"
- company: (none) -> JGY R&D
- title: (none) -> Cover Page
