File: T2601_APIArduinoExtentionBoard/T2601_APIArduinoExtentionBoard_Programmation.kicad_sch (KiCad schematic)
At the start: 12 parts

Commit message: modification organisation des dossiers
Parts:
- renumbered D to D1, D to D10, D to D26, D to D6, D to D9, J to J10, J to J11, R to R25, R to R5, R to R6, R to R7, S to S1
Changed lines of the file:
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@@
 		(dnp no)
 		(fields_autoplaced yes)
-		(property "Reference" "#PWR"
+		(property "Reference" "#PWR033"
 			(at 133.35 63.5 0)
 			(hide yes)
@@
 		(instances
 			(project "T2601_APIArduinoExtentionBoard"
-				(path "/ff48760a-7750-46de-b467-7e55c22e4653"
+				(path "/ff48760a-7750-46de-b467-7e55c22e4653/e5914230-d93f-4f7d-8e7c-6d87f4b171bf"
 					(reference "#PWR033")
 					(unit 1)
@@
 		(dnp no)
 		(fields_autoplaced yes)
-		(property "Reference" "R"
+		(property "Reference" "R7"
 			(at 30.48 45.7199 0)
 			(show_name no)
@@
 		(instances
 			(project "T2601_APIArduinoExtentionBoard"
-				(path "/ff48760a-7750-46de-b467-7e55c22e4653"
+				(path "/ff48760a-7750-46de-b467-7e55c22e4653/e5914230-d93f-4f7d-8e7c-6d87f4b171bf"
 					(reference "R7")
 					(unit 1)
@@
 		(dnp no)
 		(fields_autoplaced yes)
-		(property "Reference" "S"
+		(property "Reference" "S1"
 			(at 137.16 48.2599 90)
 			(show_name no)
@@
 		(instances
 			(project "T2601_APIArduinoExtentionBoard"
-				(path "/ff48760a-7750-46de-b467-7e55c22e4653"
+				(path "/ff48760a-7750-46de-b467-7e55c22e4653/e5914230-d93f-4f7d-8e7c-6d87f4b171bf"
 					(reference "S1")
 					(unit 1)
@@
 		(dnp no)
 		(fields_autoplaced yes)
-		(property "Reference" "#PWR"
+		(property "Reference" "#PWR039"
 			(at 33.02 74.93 0)
 			(hide yes)
@@
 		(instances
 			(project "T2601_APIArduinoExtentionBoard"
-				(path "/ff48760a-7750-46de-b467-7e55c22e4653"
+				(path "/ff48760a-7750-46de-b467-7e55c22e4653/e5914230-d93f-4f7d-8e7c-6d87f4b171bf"
 					(reference "#PWR039")
 					(unit 1)
@@
 		(dnp no)
 		(fields_autoplaced yes)
-		(property "Reference" "#PWR"
+		(property "Reference" "#PWR042"
 			(at 27.94 55.88 0)
 			(hide yes)
@@
 		(instances
 			(project "T2601_APIArduinoExtentionBoard"
-				(path "/ff48760a-7750-46de-b467-7e55c22e4653"
+				(path "/ff48760a-7750-46de-b467-7e55c22e4653/e5914230-d93f-4f7d-8e7c-6d87f4b171bf"
 					(reference "#PWR042")
 					(unit 1)
@@
 		(dnp no)
 		(fields_autoplaced yes)
-		(property "Reference" "J"
+		(property "Reference" "J11"
 			(at 78.74 46.99 90)
 			(show_name no)
@@
 		(instances
 			(project "T2601_APIArduinoExtentionBoard"
-				(path "/ff48760a-7750-46de-b467-7e55c22e4653"
+				(path "/ff48760a-7750-46de-b467-7e55c22e4653/e5914230-d93f-4f7d-8e7c-6d87f4b171bf"
 					(reference "J11")
 					(unit 1)
@@
 		(dnp no)
 		(fields_autoplaced yes)
-		(property "Reference" "#PWR"
+		(property "Reference" "#PWR043"
 			(at 38.1 55.88 0)
 			(hide yes)
@@
 		(instances
 			(project "T2601_APIArduinoExtentionBoard"
-				(path "/ff48760a-7750-46de-b467-7e55c22e4653"
+				(path "/ff48760a-7750-46de-b467-7e55c22e4653/e5914230-d93f-4f7d-8e7c-6d87f4b171bf"
 					(reference "#PWR043")
 					(unit 1)
@@
 		(dnp no)
 		(fields_autoplaced yes)
-		(property "Reference" "#PWR"
+		(property "Reference" "#PWR013"
 			(at 66.04 91.44 0)
 			(hide yes)
@@
 		(instances
 			(project "T2601_APIArduinoExtentionBoard"
-				(path "/ff48760a-7750-46de-b467-7e55c22e4653"
+				(path "/ff48760a-7750-46de-b467-7e55c22e4653/e5914230-d93f-4f7d-8e7c-6d87f4b171bf"
 					(reference "#PWR013")
 					(unit 1)
@@
 		(dnp no)
 		(fields_autoplaced yes)
-		(property "Reference" "#PWR"
+		(property "Reference" "#PWR089"
 			(at 133.35 36.83 0)
 			(hide yes)
@@
 		(instances
 			(project "T2601_APIArduinoExtentionBoard"
-				(path "/ff48760a-7750-46de-b467-7e55c22e4653"
+				(path "/ff48760a-7750-46de-b467-7e55c22e4653/e5914230-d93f-4f7d-8e7c-6d87f4b171bf"
 					(reference "#PWR089")
 					(unit 1)
@@
 		(dnp no)
 		(fields_autoplaced yes)
-		(property "Reference" "D"
+		(property "Reference" "D6"
 			(at 130.81 77.47 90)
 			(show_name no)
@@
 		(instances
 			(project "T2601_APIArduinoExtentionBoard"
-				(path "/ff48760a-7750-46de-b467-7e55c22e4653"
+				(path "/ff48760a-7750-46de-b467-7e55c22e4653/e5914230-d93f-4f7d-8e7c-6d87f4b171bf"
 					(reference "D6")
 					(unit 1)
@@
 		(dnp no)
 		(fields_autoplaced yes)
-		(property "Reference" "D"
+		(property "Reference" "D26"
 			(at 35.56 81.1846 0)
 			(show_name no)
@@
 		(instances
 			(project "T2601_APIArduinoExtentionBoard"
-				(path "/ff48760a-7750-46de-b467-7e55c22e4653"
+				(path "/ff48760a-7750-46de-b467-7e55c22e4653/e5914230-d93f-4f7d-8e7c-6d87f4b171bf"
 					(reference "D26")
 					(unit 1)
@@
 		(dnp no)
 		(fields_autoplaced yes)
-		(property "Reference" "R"
+		(property "Reference" "R25"
 			(at 35.56 74.9299 0)
 			(show_name no)
@@
 		(instances
 			(project "T2601_APIArduinoExtentionBoard"
-				(path "/ff48760a-7750-46de-b467-7e55c22e4653"
+				(path "/ff48760a-7750-46de-b467-7e55c22e4653/e5914230-d93f-4f7d-8e7c-6d87f4b171bf"
 					(reference "R25")
 					(unit 1)
@@
 		(dnp no)
 		(fields_autoplaced yes)
-		(property "Reference" "D"
+		(property "Reference" "D10"
 			(at 40.64 36.7346 0)
 			(show_name no)
@@
 		(instances
 			(project "T2601_APIArduinoExtentionBoard"
-				(path "/ff48760a-7750-46de-b467-7e55c22e4653"
+				(path "/ff48760a-7750-46de-b467-7e55c22e4653/e5914230-d93f-4f7d-8e7c-6d87f4b171bf"
 					(reference "D10")
 					(unit 1)
@@
 		(in_pos_files yes)
 		(dnp no)
-		(property "Reference" "J"
+		(property "Reference" "J10"
 			(at 83.82 72.39 0)
 			(show_name no)
@@
 		(instances
 			(project "T2601_APIArduinoExtentionBoard"
-				(path "/ff48760a-7750-46de-b467-7e55c22e4653"
+				(path "/ff48760a-7750-46de-b467-7e55c22e4653/e5914230-d93f-4f7d-8e7c-6d87f4b171bf"
 					(reference "J10")
 					(unit 1)
@@
 		(dnp no)
 		(fields_autoplaced yes)
-		(property "Reference" "#PWR"
+		(property "Reference" "#PWR019"
 			(at 87.63 46.99 0)
 			(hide yes)
@@
 		(instances
 			(project "T2601_APIArduinoExtentionBoard"
-				(path "/ff48760a-7750-46de-b467-7e55c22e4653"
+				(path "/ff48760a-7750-46de-b467-7e55c22e4653/e5914230-d93f-4f7d-8e7c-6d87f4b171bf"
 					(reference "#PWR019")
 					(unit 1)
@@
 		(dnp no)
 		(fields_autoplaced yes)
-		(property "Reference" "R"
+		(property "Reference" "R5"
 			(at 128.27 38.0999 0)
 			(show_name no)
@@
 		(instances
 			(project "T2601_APIArduinoExtentionBoard"
-				(path "/ff48760a-7750-46de-b467-7e55c22e4653"
+				(path "/ff48760a-7750-46de-b467-7e55c22e4653/e5914230-d93f-4f7d-8e7c-6d87f4b171bf"
 					(reference "R5")
 					(unit 1)
@@
 		(dnp no)
 		(fields_autoplaced yes)
-		(property "Reference" "D"
+		(property "Reference" "D1"
 			(at 69.85 69.5324 90)
 			(show_name no)
@@
 		(instances
 			(project "T2601_APIArduinoExtentionBoard"
-				(path "/ff48760a-7750-46de-b467-7e55c22e4653"
+				(path "/ff48760a-7750-46de-b467-7e55c22e4653/e5914230-d93f-4f7d-8e7c-6d87f4b171bf"
 					(reference "D1")
 					(unit 1)
@@
 		(dnp no)
 		(fields_autoplaced yes)
-		(property "Reference" "R"
+		(property "Reference" "R6"
 			(at 40.64 45.7199 0)
 			(show_name no)
@@
 		(instances
 			(project "T2601_APIArduinoExtentionBoard"
-				(path "/ff48760a-7750-46de-b467-7e55c22e4653"
+				(path "/ff48760a-7750-46de-b467-7e55c22e4653/e5914230-d93f-4f7d-8e7c-6d87f4b171bf"
 					(reference "R6")
 					(unit 1)
@@
 		(dnp no)
 		(fields_autoplaced yes)
-		(property "Reference" "D"
+		(property "Reference" "D9"
 			(at 30.48 36.7346 0)
 			(show_name no)
@@
 		(instances
 			(project "T2601_APIArduinoExtentionBoard"
-				(path "/ff48760a-7750-46de-b467-7e55c22e4653"
+				(path "/ff48760a-7750-46de-b467-7e55c22e4653/e5914230-d93f-4f7d-8e7c-6d87f4b171bf"
 					(reference "D9")
 					(unit 1)
@@
 		(dnp no)
 		(fields_autoplaced yes)
-		(property "Reference" "#PWR"
+		(property "Reference" "#PWR014"
 			(at 67.31 71.12 0)
 			(hide yes)
@@
 		(instances
 			(project "T2601_APIArduinoExtentionBoard"
-				(path "/ff48760a-7750-46de-b467-7e55c22e4653"
+				(path "/ff48760a-7750-46de-b467-7e55c22e4653/e5914230-d93f-4f7d-8e7c-6d87f4b171bf"
 					(reference "#PWR014")
 					(unit 1)
@@
 		(dnp no)
 		(fields_autoplaced yes)
-		(property "Reference" "#PWR"
+		(property "Reference" "#PWR029"
 			(at 125.73 38.1 0)
 			(hide yes)
@@
 		(instances
 			(project "T2601_APIArduinoExtentionBoard"
-				(path "/ff48760a-7750-46de-b467-7e55c22e4653"
+				(path "/ff48760a-7750-46de-b467-7e55c22e4653/e5914230-d93f-4f7d-8e7c-6d87f4b171bf"
 					(reference "#PWR029")
 					(unit 1)
