File: T2601_APIArduinoExtentionBoard/T2601_MCU_Prog.kicad_sch (KiCad schematic)
At the start: 6 parts

Commit message: Test point GND
Parts:
- renumbered D to D52, D to D54, D to D55, J to J28, R to R51, R to R53
Changed lines of the file:
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@@
 		(dnp no)
 		(fields_autoplaced yes)
-		(property "Reference" "#PWR"
+		(property "Reference" "#PWR0182"
 			(at 119.38 85.09 0)
 			(hide yes)
@@
 		(instances
 			(project "T2601_APIArduinoExtentionBoard"
-				(path "/ff48760a-7750-46de-b467-7e55c22e4653/fede4c36-00cc-4d3d-b71c-5243ba232202"
+				(path "/ff48760a-7750-46de-b467-7e55c22e4653/fede4c36-00cc-4d3d-b71c-5243ba232202/24664caa-e0c0-4ea4-b2a3-fac74f670bd6"
 					(reference "#PWR0182")
 					(unit 1)
@@
 		(dnp no)
 		(fields_autoplaced yes)
-		(property "Reference" "R"
+		(property "Reference" "R51"
 			(at 176.53 95.2499 0)
 			(show_name no)
@@
 		(instances
 			(project "T2601_APIArduinoExtentionBoard"
-				(path "/ff48760a-7750-46de-b467-7e55c22e4653/fede4c36-00cc-4d3d-b71c-5243ba232202"
+				(path "/ff48760a-7750-46de-b467-7e55c22e4653/fede4c36-00cc-4d3d-b71c-5243ba232202/24664caa-e0c0-4ea4-b2a3-fac74f670bd6"
 					(reference "R51")
 					(unit 1)
@@
 		(dnp no)
 		(fields_autoplaced yes)
-		(property "Reference" "R"
+		(property "Reference" "R53"
 			(at 186.69 95.2499 0)
 			(show_name no)
@@
 		(instances
 			(project "T2601_APIArduinoExtentionBoard"
-				(path "/ff48760a-7750-46de-b467-7e55c22e4653/fede4c36-00cc-4d3d-b71c-5243ba232202"
+				(path "/ff48760a-7750-46de-b467-7e55c22e4653/fede4c36-00cc-4d3d-b71c-5243ba232202/24664caa-e0c0-4ea4-b2a3-fac74f670bd6"
 					(reference "R53")
 					(unit 1)
@@
 		(dnp no)
 		(fields_autoplaced yes)
-		(property "Reference" "D"
+		(property "Reference" "D54"
 			(at 186.69 86.2646 0)
 			(show_name no)
@@
 		(instances
 			(project "T2601_APIArduinoExtentionBoard"
-				(path "/ff48760a-7750-46de-b467-7e55c22e4653/fede4c36-00cc-4d3d-b71c-5243ba232202"
+				(path "/ff48760a-7750-46de-b467-7e55c22e4653/fede4c36-00cc-4d3d-b71c-5243ba232202/24664caa-e0c0-4ea4-b2a3-fac74f670bd6"
 					(reference "D54")
 					(unit 1)
@@
 		(in_pos_files yes)
 		(dnp no)
-		(property "Reference" "J"
+		(property "Reference" "J28"
 			(at 136.144 100.838 0)
 			(show_name no)
@@
 		(instances
 			(project "T2601_APIArduinoExtentionBoard"
-				(path "/ff48760a-7750-46de-b467-7e55c22e4653/fede4c36-00cc-4d3d-b71c-5243ba232202"
+				(path "/ff48760a-7750-46de-b467-7e55c22e4653/fede4c36-00cc-4d3d-b71c-5243ba232202/24664caa-e0c0-4ea4-b2a3-fac74f670bd6"
 					(reference "J28")
 					(unit 1)
@@
 		(dnp no)
 		(fields_autoplaced yes)
-		(property "Reference" "D"
+		(property "Reference" "D52"
 			(at 176.53 86.2646 0)
 			(show_name no)
@@
 		(instances
 			(project "T2601_APIArduinoExtentionBoard"
-				(path "/ff48760a-7750-46de-b467-7e55c22e4653/fede4c36-00cc-4d3d-b71c-5243ba232202"
+				(path "/ff48760a-7750-46de-b467-7e55c22e4653/fede4c36-00cc-4d3d-b71c-5243ba232202/24664caa-e0c0-4ea4-b2a3-fac74f670bd6"
 					(reference "D52")
 					(unit 1)
@@
 		(dnp no)
 		(fields_autoplaced yes)
-		(property "Reference" "#PWR"
+		(property "Reference" "#PWR0181"
 			(at 118.11 105.41 0)
 			(hide yes)
@@
 		(instances
 			(project "T2601_APIArduinoExtentionBoard"
-				(path "/ff48760a-7750-46de-b467-7e55c22e4653/fede4c36-00cc-4d3d-b71c-5243ba232202"
+				(path "/ff48760a-7750-46de-b467-7e55c22e4653/fede4c36-00cc-4d3d-b71c-5243ba232202/24664caa-e0c0-4ea4-b2a3-fac74f670bd6"
 					(reference "#PWR0181")
 					(unit 1)
@@
 		(dnp no)
 		(fields_autoplaced yes)
-		(property "Reference" "D"
+		(property "Reference" "D55"
 			(at 121.92 83.5024 90)
 			(show_name no)
@@
 		(instances
 			(project "T2601_APIArduinoExtentionBoard"
-				(path "/ff48760a-7750-46de-b467-7e55c22e4653/fede4c36-00cc-4d3d-b71c-5243ba232202"
+				(path "/ff48760a-7750-46de-b467-7e55c22e4653/fede4c36-00cc-4d3d-b71c-5243ba232202/24664caa-e0c0-4ea4-b2a3-fac74f670bd6"
 					(reference "D55")
 					(unit 1)
@@
 		(dnp no)
 		(fields_autoplaced yes)
-		(property "Reference" "#PWR"
+		(property "Reference" "#PWR0180"
 			(at 184.15 105.41 0)
 			(hide yes)
@@
 		(instances
 			(project "T2601_APIArduinoExtentionBoard"
-				(path "/ff48760a-7750-46de-b467-7e55c22e4653/fede4c36-00cc-4d3d-b71c-5243ba232202"
+				(path "/ff48760a-7750-46de-b467-7e55c22e4653/fede4c36-00cc-4d3d-b71c-5243ba232202/24664caa-e0c0-4ea4-b2a3-fac74f670bd6"
 					(reference "#PWR0180")
 					(unit 1)
@@
 		(dnp no)
 		(fields_autoplaced yes)
-		(property "Reference" "#PWR"
+		(property "Reference" "#PWR0178"
 			(at 173.99 105.41 0)
 			(hide yes)
@@
 		(instances
 			(project "T2601_APIArduinoExtentionBoard"
-				(path "/ff48760a-7750-46de-b467-7e55c22e4653/fede4c36-00cc-4d3d-b71c-5243ba232202"
+				(path "/ff48760a-7750-46de-b467-7e55c22e4653/fede4c36-00cc-4d3d-b71c-5243ba232202/24664caa-e0c0-4ea4-b2a3-fac74f670bd6"
 					(reference "#PWR0178")
 					(unit 1)

Commit message: Reroutage en cours 2
Connections:
- net MISO: now also J28.3 (Pin_3); no longer J28.5 (Pin_5)
- net MOSI: now also J28.5 (Pin_5); no longer J28.3 (Pin_3)
Changed lines of the file:
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@@
 	(global_label "MISO"
 		(shape input)
-		(at 142.24 95.25 0)
+		(at 129.54 97.79 180)
 		(fields_autoplaced yes)
 		(effects
@@
 				(size 1.27 1.27)
 			)
-			(justify left)
+			(justify right)
 		)
 		(property "Intersheetrefs" "${INTERSHEET_REFS}"
-			(at 149.8214 95.25 0)
+			(at 122.3341 97.79 0)
 			(hide yes)
 			(show_name no)
@@
 					(size 1.27 1.27)
 				)
-				(justify left)
+				(justify right)
 			)
 		)
@@
 	(global_label "MOSI"
 		(shape input)
-		(at 129.54 97.79 180)
+		(at 142.24 95.25 0)
 		(fields_autoplaced yes)
 		(effects
@@
 				(size 1.27 1.27)
 			)
-			(justify right)
+			(justify left)
 		)
 		(property "Intersheetrefs" "${INTERSHEET_REFS}"
-			(at 121.9586 97.79 0)
+			(at 149.4459 95.25 0)
 			(hide yes)
 			(show_name no)
@@
 					(size 1.27 1.27)
 				)
-				(justify right)
+				(justify left)
 			)
 		)

Commit message: Rerouting done
Connections:
- net GND: now also D52.1, D54.1; no longer R51.2, R53.2
- net MISO: now also R53.1; no longer D54.2
- net MOSI: now also R51.1; no longer D52.2
- new net: D52.2, R51.2
- new net: D54.2, R53.2
Other:
- moved on the sheet: D52, D54, R51, R53
