File: T2601_APIArduinoExtentionBoard/T2601_Power.kicad_sch (KiCad schematic)
At the start: 20 parts, among them J24 Conn_01x04_Pin, J25 Conn_01x04_Pin

Commit message: correction DRC
Parts:
- removed JP15, JP19, JP23: SolderJumper_2_Open, Jumper:SolderJumper-2_P1.3mm_Open_RoundedPad1.0x1.5mm, symbol Jumper:SolderJumper_2_Open
